Commit message: ad_r1m_perception_cuvslam, pointcloud_to_occupancygrid: Tune multi-camera config
Update cuVSLAM multi-realsense launch and config for dual-camera
setup, adjust calibration URDF, and tune occupancy grid build params.

Signed-off-by: Tudor Alinei-Poiana <tudor.alinei-poiana@analog.com>

File: ad_r1m_perception_cuvslam/urdf/realsense_calibration.urdf.xacro (robot description, xacro)
@@ -5,5 +5,5 @@
     <parent link="base_link"/>
     <child link="camera1_link"/>
-    <origin xyz="0.0 0.0 0.0" rpy="0 0 0"/>
+    <origin xyz="0.3 0.0 0.0" rpy="0 0 0"/>
   </joint>
   <link name="camera1_link"/>
@@ -11,5 +11,6 @@
     <parent link="base_link"/>
     <child link="camera2_link"/>
-    <origin xyz="-0.14 0.06 0.0" rpy="0 0 -1.5707"/>
+    <!--origin xyz="-0.098 -0.032 0.0" rpy="0 0 -1.5707"/-->
+    <origin xyz="-0.048876 -0.055130 0.032332" rpy="0.028781 0.000890 -1.583501"/>
   </joint>
   <link name="camera2_link"/>
