Commit message: ad_r1m_description: Fix wheel slip and odometry drift in Gazebo sim
Change drive wheel collision from sphere to cylinder in order to have collision and visual matched. Add ODE contact parameters (kp, kd, minDepth, maxVel) to all
wheels. Increase wheel mass from 0.05 to
0.5 kg to make simulation parameters resemble the real system. Reduce drive wheel friction
coefficients from 2.5 to 1.5 (this might make the solver more stable).

Add wheel_separation property (0.29 m) matching the diff_drive_controller
config and use it for drive wheel placement instead of base_width, fixing
a odometry rotation underestimate (Gazebo robot was turning more than what the diff_drive_controller was computig due to this mismatch between the robot description and controller parameters).

All new lines are tagged with SLIP_FIX comments for easy identification.

Signed-off-by: Tudor Alinei-Poiana <tudor.alinei-poiana@analog.com>

File: ad_r1m_description/urdf/ad_r1m_base.urdf.xacro (robot description, xacro)
@@ -10,9 +10,10 @@
     <xacro:property name="chassis_height" value="0.15"/>
     <xacro:property name="base_width" value="0.22"/>
+    <xacro:property name="wheel_separation" value="0.29"/>
     <xacro:property name="chassis_zoff" value="0.08"/>
     <xacro:property name="chassis_mass" value="1.0"/>
     <xacro:property name="wheel_radius" value="0.05"/>
     <xacro:property name="wheel_width" value="0.025"/>
-    <xacro:property name="wheel_mass" value="0.05"/>
+    <xacro:property name="wheel_mass" value="0.5"/> <!-- SLIP_FIX was 0.05 -->
     <xacro:property name="caster_wheel_radius" value="0.025"/>
     <xacro:property name="caster_wheel_mass" value="0.01"/>
@@ -75,5 +76,5 @@
         <parent link="${prefix}base_link"/>
         <child link="${prefix}left_wheel"/>
-        <origin xyz="0 ${(base_width + wheel_width)/2} ${wheel_radius}" rpy="-${pi/2} 0 0" />
+        <origin xyz="0 ${wheel_separation/2} ${wheel_radius}" rpy="-${pi/2} 0 0" />
         <axis xyz="0 0 1"/>
     </joint>
@@ -87,5 +88,5 @@
         <collision>
             <geometry>
-                <sphere radius="${wheel_radius}"/>
+                <cylinder radius="${wheel_radius}" length="${wheel_width}"/> <!-- SLIP_FIX was sphere -->
             </geometry>
         </collision>
@@ -96,6 +97,10 @@
     <gazebo reference="${prefix}left_wheel">
         <material>Gazebo/Black</material>
-        <mu1>2.5</mu1>
-        <mu2>2.5</mu2>
+        <mu1>1.5</mu1> <!-- SLIP_FIX was 2.5 -->
+        <mu2>1.5</mu2> <!-- SLIP_FIX was 2.5 -->
+        <kp>1000000</kp> <!-- SLIP_FIX -->
+        <kd>100</kd> <!-- SLIP_FIX -->
+        <minDepth>0.001</minDepth> <!-- SLIP_FIX -->
+        <maxVel>0.1</maxVel> <!-- SLIP_FIX -->
     </gazebo>
     <!-- RIGHT WHEEL LINK -->
@@ -103,5 +108,5 @@
         <parent link="${prefix}base_link"/>
         <child link="${prefix}right_wheel"/>
-        <origin xyz="0 ${-(base_width + wheel_width)/2} ${wheel_radius}" rpy="${pi/2} 0 0" />
+        <origin xyz="0 ${-wheel_separation/2} ${wheel_radius}" rpy="${pi/2} 0 0" />
         <axis xyz="0 0 -1"/>
     </joint>
@@ -115,5 +120,5 @@
         <collision>
             <geometry>
-                <sphere radius="${wheel_radius}"/>
+                <cylinder radius="${wheel_radius}" length="${wheel_width}"/> <!-- SLIP_FIX was sphere -->
             </geometry>
         </collision>
@@ -124,6 +129,10 @@
     <gazebo reference="${prefix}right_wheel">
         <material>Gazebo/Black</material>
-        <mu1>2.5</mu1>
-        <mu2>2.5</mu2>
+        <mu1>1.5</mu1> <!-- SLIP_FIX was 2.5 -->
+        <mu2>1.5</mu2> <!-- SLIP_FIX was 2.5 -->
+        <kp>1000000</kp> <!-- SLIP_FIX -->
+        <kd>100</kd> <!-- SLIP_FIX -->
+        <minDepth>0.001</minDepth> <!-- SLIP_FIX -->
+        <maxVel>0.1</maxVel> <!-- SLIP_FIX -->
     </gazebo>
     <!-- CASTER WHEEL LINKS -->
@@ -155,4 +164,8 @@
             <mu1 value="0.001"/>
             <mu2 value="0.001"/>
+            <kp>1000000</kp> <!-- SLIP_FIX -->
+            <kd>100</kd> <!-- SLIP_FIX -->
+            <minDepth>0.001</minDepth> <!-- SLIP_FIX -->
+            <maxVel>0.1</maxVel> <!-- SLIP_FIX -->
         </gazebo>
     </xacro:macro>

Commit message: ad_r1m_description: Fix stacked visual offset in chassis URDF
The chassis_zoff was applied twice, once in the joint origin and again
in the visual/collision/inertial origins. Workaorund was dividing offset by 2.
Removed the redundant offset from visual, collision, and inertial elements,
positioned the chassis joint correctly at z_offset = ground_clearance + height/2.

Signed-off-by: laurent-19 <laurentiu.popa@analog.com>

File: ad_r1m_description/urdf/ad_r1m_base.urdf.xacro (robot description, xacro)
@@ -12,5 +12,5 @@
     <xacro:property name="wheel_separation" value="0.29"/>
     <xacro:property name="chassis_clearance_ground" value="0.010"/>
-    <xacro:property name="chassis_zoff" value="${(chassis_clearance_ground + chassis_height/2) / 2}"/>
+    <xacro:property name="chassis_zoff" value="${(chassis_clearance_ground + chassis_height/2)}"/>
     <xacro:property name="chassis_mass" value="1.0"/>
     <xacro:property name="wheel_radius" value="0.05"/>
@@ -58,5 +58,4 @@
     <link name="${prefix}chassis">
         <visual>
-            <origin xyz="0 0 ${chassis_zoff}"/>
             <geometry>
                 <box size="${chassis_length} ${chassis_width} ${chassis_height}"/>
@@ -65,5 +64,4 @@
         </visual>
         <collision>
-            <origin xyz="0 0 ${chassis_zoff}"/>
             <geometry>
                 <box size="${chassis_length} ${chassis_width} ${chassis_height}"/>
@@ -71,5 +69,5 @@
         </collision>
         <xacro:inertial_box mass="10.0" x="${chassis_length}" y="${chassis_width}" z="${chassis_height}">
-            <origin xyz="0 0 ${chassis_zoff}" rpy="0 0 0"/>
+            <origin xyz="0 0 0" rpy="0 0 0"/>
         </xacro:inertial_box>
     </link>
@@ -83,5 +81,5 @@
             <parent link="${prefix}chassis"/>
             <child link="${prefix}${name}_bumper_lat"/>
-            <origin xyz="${x_reflect*(chassis_length/2 - bumper_length/2)} ${y_reflect*(chassis_width/2 + bumper_thickness/2)} ${chassis_zoff}" rpy="0 0 0"/>
+	    <origin xyz="${x_reflect*(chassis_length/2 - bumper_length/2)} ${y_reflect*(chassis_width/2 + bumper_thickness/2)} 0" rpy="0 0 0"/>
         </joint>
         <link name="${prefix}${name}_bumper_lat">
@@ -100,5 +98,5 @@
             <parent link="${prefix}chassis"/>
             <child link="${prefix}${name}_bumper_front"/>
-            <origin xyz="${x_reflect*(chassis_length/2 + bumper_thickness/2)} ${y_reflect*(chassis_width/2 - bumper_length/2 + bumper_thickness/2)} ${chassis_zoff}" rpy="0 0 0"/>
+	    <origin xyz="${x_reflect*(chassis_length/2 + bumper_thickness/2)} ${y_reflect*(chassis_width/2 - bumper_length/2 + bumper_thickness/2)} 0" rpy="0 0 0"/>
         </joint>
         <link name="${prefix}${name}_bumper_front">
