Commit message: ad_r1m_description: Fix ToF camera simulation to match real hardware
ToF Camera (_tof_adtf3175d.xacro):
- Change sensor type from 'camera' to 'depth' for proper depth output
- Fix FOV from 114deg to 75deg (1.309 rad) per ADTF3175D datasheet
- Fix optical frame rotation to match real driver (-pi/2, 0, -pi/2)
- Add 5mm Gaussian noise to match sensor accuracy spec
- Update depth range to 0.3-5.0m per depth_to_laser_params.yaml
- Remap topics to match real robot: ab_image, depth_image, point_cloud
- Update rate from 10Hz to 30Hz

Lidar (_lidar.xacro):
- Use cam1_scan frame instead of cam1_laser (matches depthimage_to_laserscan)
- Update samples from 75 to 512 (matches image width)
- Update range to 0.3-5.0m
- Use relative topic remapping for proper namespacing

Signed-off-by: laurent-19 <laurentiu.popa@analog.com>

File: ad_r1m_description/urdf/_lidar.xacro (robot description, xacro)
@@ -1,55 +1,32 @@
 <?xml version="1.0"?>
 <robot xmlns:xacro="http://www.ros.org/wiki/xacro" >
+<!-- Simulated 2D laser scan - mimics depthimage_to_laserscan output.
+     Reuses cam1_scan frame from _tof_adtf3175d.xacro.
+     75deg FOV, 0.3-5.0m range -->
 <xacro:macro name="lidar" params="prefix parent *origin">
-    <joint name="cam1_laser_joint" type="fixed">
-        <parent link="${parent}"/>
-        <child link="${prefix}cam1_laser"/>
-        <xacro:insert_block name="origin" />
-    </joint>
-    <link name="${prefix}cam1_laser">
-        <inertial>
-            <origin xyz="0 0 0" rpy="0 0 0"/>
-            <mass value="0.125"/>
-            <inertia ixx="0.001" ixy="0" ixz="0" iyy="0.001" iyz="0" izz="0.001" />
-        </inertial>
-        <collision>
-            <origin xyz="0 0 0" rpy="0 0 0"/>
-            <geometry>
-                <box size="0.065 0.075 0.05"/>
-            </geometry>
-        </collision>
-        <visual>
-            <origin xyz="0 0 0" rpy="0 0 0"/>
-            <geometry>
-                <box size="0.065 0.075 0.05"/>
-            </geometry>
-            <material name="black"/>
-        </visual>
-    </link>
-    <gazebo reference="${prefix}cam1_laser">
-        <material>Gazebo/Black</material>
+    <gazebo reference="${prefix}cam1_scan">
         <sensor name="laser" type="ray">
-            <pose> 0 0 0 0 0 0 </pose>
+            <pose>0 0 0 0 0 0</pose>
             <visualize>false</visualize>
-            <update_rate>10</update_rate>
+            <update_rate>30</update_rate>
             <ray>
                 <scan>
                     <horizontal>
-                        <samples>75</samples>
-                        <min_angle>-0.654166</min_angle>
-                        <max_angle>0.654166</max_angle>
+                        <samples>512</samples>
+                        <min_angle>-0.6545</min_angle>
+                        <max_angle>0.6545</max_angle>
                     </horizontal>
                 </scan>
                 <range>
-                    <min>0.4</min>
-                    <max>5</max>
+                    <min>0.3</min>
+                    <max>5.0</max>
                 </range>
             </ray>
             <plugin name="laser_controller" filename="libgazebo_ros_ray_sensor.so">
                 <ros>
-                    <remapping>~/out:=/scan</remapping>
+                    <remapping>~/out:=scan</remapping>
                 </ros>
                 <output_type>sensor_msgs/LaserScan</output_type>
-                <frame_name>cam1_laser</frame_name>
+                <frame_name>${prefix}cam1_scan</frame_name>
             </plugin>
         </sensor>

File: ad_r1m_description/urdf/_tof_adtf3175d.xacro (robot description, xacro)
@@ -30,5 +30,5 @@
         <parent link="${prefix}cam1_adtf31xx"/>
         <child link="${prefix}cam1_adtf31xx_optical"/>
-        <origin xyz="0 0 0" rpy="${pi/2} 0 ${pi/2}"/>
+        <origin xyz="0 0 0" rpy="${-pi/2} 0 ${-pi/2}"/>
     </joint>
     <link name="${prefix}cam1_adtf31xx_optical"></link>
@@ -41,22 +41,36 @@
     <gazebo reference="${prefix}cam1_adtf31xx">
         <material>Gazebo/Black</material>
-        <sensor name="${prefix}cam1" type="camera">
-            <pose> 0 0 0 0 0 0 </pose>
+        <!-- ADTF3175D ToF Camera - 75deg FOV, 512x512, 0.3-5.0m range -->
+        <sensor name="cam1_depth" type="depth">
+            <pose>0 0 0 0 0 0</pose>
             <visualize>true</visualize>
-            <update_rate>10</update_rate>
+            <update_rate>30</update_rate>
             <camera>
-                <horizontal_fov>2</horizontal_fov>
+                <horizontal_fov>1.309</horizontal_fov>
                 <image>
-                    <format>BGR8</format>
                     <width>512</width>
                     <height>512</height>
+                    <format>R8G8B8</format>
                 </image>
                 <clip>
-                    <near>0.4</near>
+                    <near>0.3</near>
                     <far>5.0</far>
                 </clip>
+                <noise>
+                    <type>gaussian</type>
+                    <mean>0.0</mean>
+                    <stddev>0.005</stddev>
+                </noise>
             </camera>
-            <plugin name="camera_controller" filename="libgazebo_ros_camera.so">
+            <plugin name="depth_camera_controller" filename="libgazebo_ros_camera.so">
+                <camera_name>cam1</camera_name>
                 <frame_name>${prefix}cam1_adtf31xx_optical</frame_name>
+                <min_depth>0.1</min_depth>
+                <max_depth>10.0</max_depth>
+                <ros>
+                    <remapping>cam1/image_raw:=cam1/ab_image</remapping>
+                    <remapping>cam1/depth/image_raw:=cam1/depth_image</remapping>
+                    <remapping>cam1/points:=cam1/point_cloud</remapping>
+                </ros>
             </plugin>
         </sensor>
