Commit message: ad_r1m_description: Align ToF depth range and update RViz config
ToF Camera (_tof_adtf3175d.xacro):
- Align min/max depth to 0.3-5.0m (matches camera clip range)
- Add use_sim parameter for optical frame rotation:
  - sim: -pi/2
  - real: +pi/2 (real depth image is flipped vs gazebo depth)
- Document simulation vs real hardware differences

RViz (main_sim.rviz):
- Add depth_image display with correct settings for 32FC1
- Add point_cloud display for ToF visualization
- Update ab_image topic from image_raw

Signed-off-by: laurent-19 <laurentiu.popa@analog.com>

File: ad_r1m_description/urdf/_tof_adtf3175d.xacro (robot description, xacro)
@@ -1,5 +1,14 @@
 <?xml version="1.0"?>
-<robot xmlns:xacro="http://www.ros.org/wiki/xacro" >
-<xacro:macro name="tof_adtf3175d" params="prefix parent *origin">
+<!--
+  ADTF3175D ToF Camera
+  Simulation vs Real Hardware differences:
+    - depth_image: 32FC1 in meters (real: 16UC1 in mm)
+    - point_cloud: XYZRGB fields (real: XYZ only)
+    - optical_frame: sim uses -pi/2 (Gazebo), real uses pi/2 (driver flips image)
+-->
+<robot xmlns:xacro="http://www.ros.org/wiki/xacro">
+<xacro:macro name="tof_adtf3175d" params="prefix parent use_sim:=false *origin">
+    <!-- Optical frame rotation differs: real driver flips image internally -->
+    <xacro:property name="optical_sign" value="${-1 if use_sim else 1}"/>
     <joint name="cam1_adtf31xx_joint" type="fixed">
         <parent link="${parent}"/>
@@ -30,16 +39,16 @@
         <parent link="${prefix}cam1_adtf31xx"/>
         <child link="${prefix}cam1_adtf31xx_optical"/>
-        <origin xyz="0 0 0" rpy="${-pi/2} 0 ${-pi/2}"/>
+        <origin xyz="0 0 0" rpy="${optical_sign * pi/2} 0 ${optical_sign * pi/2}"/>
     </joint>
     <link name="${prefix}cam1_adtf31xx_optical"></link>
     <joint name="cam1_scan_joint" type="fixed">
-	    <parent link="${prefix}cam1_adtf31xx"/>
-	    <child link="${prefix}cam1_scan"/>
-		<origin xyz="0 0 0" rpy="${pi} 0 0" />
-	</joint>
-	<link name="${prefix}cam1_scan"></link>
+        <parent link="${prefix}cam1_adtf31xx"/>
+        <child link="${prefix}cam1_scan"/>
+        <origin xyz="0 0 0" rpy="${pi} 0 0"/>
+    </joint>
+    <link name="${prefix}cam1_scan"></link>
     <gazebo reference="${prefix}cam1_adtf31xx">
         <material>Gazebo/Black</material>
-        <!-- ADTF3175D ToF Camera - 75deg FOV, 512x512, 0.3-5.0m range -->
+        <!-- 75deg FOV, 512x512, 0.3-5.0m range -->
         <sensor name="cam1_depth" type="depth">
             <pose>0 0 0 0 0 0</pose>
@@ -66,6 +75,6 @@
                 <camera_name>cam1</camera_name>
                 <frame_name>${prefix}cam1_adtf31xx_optical</frame_name>
-                <min_depth>0.1</min_depth>
-                <max_depth>10.0</max_depth>
+                <min_depth>0.3</min_depth>
+                <max_depth>5.0</max_depth>
                 <ros>
                     <remapping>cam1/image_raw:=cam1/ab_image</remapping>

File: ad_r1m_description/urdf/ad_r1m_base.urdf.xacro (robot description, xacro)
@@ -5,5 +5,5 @@
 <xacro:include filename="_tof_adtf3175d.xacro" />
 <xacro:include filename="_imu_adis16470.xacro" />
-<xacro:macro name="ad_r1m_base" params="prefix">
+<xacro:macro name="ad_r1m_base" params="prefix use_sim:=false">
     <xacro:property name="chassis_length" value="0.59"/>
     <xacro:property name="chassis_width" value="0.36"/>
@@ -37,5 +37,5 @@
         <origin xyz="0.180 0 ${wheel_radius}" rpy="${pi} 0 ${-pi/2}"/>
     </xacro:imu_adis16470>
-    <xacro:tof_adtf3175d prefix="${prefix}" parent="${prefix}base_link">
+    <xacro:tof_adtf3175d prefix="${prefix}" parent="${prefix}base_link" use_sim="${use_sim}">
         <origin xyz="${chassis_length/2 + camera_overhang - camera_length/2} 0 ${chassis_clearance_ground + camera_offset_above_chassis + camera_height/2}" rpy="0 0 0" />
     </xacro:tof_adtf3175d>

File: ad_r1m_gazebo/urdf/ad_r1m_sim.urdf.xacro (robot description, xacro)
@@ -10,5 +10,5 @@
     <!-- Instantiate base robot model -->
     <xacro:include filename="$(find ad_r1m_description)/urdf/ad_r1m_base.urdf.xacro" />
-    <xacro:ad_r1m_base prefix="${prefix}" />
+    <xacro:ad_r1m_base prefix="${prefix}" use_sim="true" />
     <!-- Bind gazebo_ros2_control to previously defined joints (e.g. left_wheel_joint) -->
     <ros2_control name="GazeboSystem" type="system">
