Commit message: Update URDF model to match physical robot dimensions and colors
- Fix wheel heights: caster wheels now level with drive wheels
- Update chassis dimensions (0.59x0.36x0.12m) and ground clearance (10mm)
- Add ADI color scheme: white chassis, gray wheels, blue corner bumpers
- Add L-shaped corner bumpers at all four corners
- Fix camera/lidar positioning with parameterized offsets
- Match ToF camera and lidar geometry to actual sensor size (65x75x50mm)
- Define IMU material inline to fix undefined material warning

Signed-off-by: laurent-19 <laurentiu.popa@analog.com>

File: ad_r1m_description/urdf/_imu_adis16470.xacro (robot description, xacro)
@@ -24,5 +24,7 @@
                 <box size="0.015 0.01 0.01"/>
             </geometry>
-            <material name="white" />
+            <material name="white">
+                <color rgba="1 1 1 1"/>
+            </material>
         </visual>
     </link>

File: ad_r1m_description/urdf/_lidar.xacro (robot description, xacro)
@@ -16,5 +16,5 @@
             <origin xyz="0 0 0" rpy="0 0 0"/>
             <geometry>
-                <box size="0.02 0.065 0.07"/>
+                <box size="0.065 0.075 0.05"/>
             </geometry>
         </collision>
@@ -22,5 +22,5 @@
             <origin xyz="0 0 0" rpy="0 0 0"/>
             <geometry>
-                <box size="0.02 0.065 0.07"/>
+                <box size="0.065 0.075 0.05"/>
             </geometry>
             <material name="black"/>

File: ad_r1m_description/urdf/_tof_adtf3175d.xacro (robot description, xacro)
@@ -16,5 +16,5 @@
             <origin xyz="0 0 0" rpy="0 0 0"/>
             <geometry>
-                <box size="0.02 0.065 0.07"/>
+                <box size="0.065 0.075 0.05"/>
             </geometry>
         </collision>
@@ -22,5 +22,5 @@
             <origin xyz="0 0 0" rpy="0 0 0"/>
             <geometry>
-                <box size="0.02 0.065 0.07"/>
+                <box size="0.065 0.075 0.05"/>
             </geometry>
             <material name="black"/>

File: ad_r1m_description/urdf/ad_r1m_base.urdf.xacro (robot description, xacro)
@@ -6,10 +6,11 @@
 <xacro:include filename="_imu_adis16470.xacro" />
 <xacro:macro name="ad_r1m_base" params="prefix">
-    <xacro:property name="chassis_length" value="0.585"/>
+    <xacro:property name="chassis_length" value="0.59"/>
     <xacro:property name="chassis_width" value="0.36"/>
-    <xacro:property name="chassis_height" value="0.15"/>
+    <xacro:property name="chassis_height" value="0.12"/>
     <xacro:property name="base_width" value="0.22"/>
     <xacro:property name="wheel_separation" value="0.29"/>
-    <xacro:property name="chassis_zoff" value="0.08"/>
+    <xacro:property name="chassis_clearance_ground" value="0.010"/>
+    <xacro:property name="chassis_zoff" value="${(chassis_clearance_ground + chassis_height/2) / 2}"/>
     <xacro:property name="chassis_mass" value="1.0"/>
     <xacro:property name="wheel_radius" value="0.05"/>
@@ -18,12 +19,16 @@
     <xacro:property name="caster_wheel_radius" value="0.025"/>
     <xacro:property name="caster_wheel_mass" value="0.01"/>
-    <xacro:property name="caster_wheel_zoff" value="${caster_wheel_radius + 0.005}"/>
-    <material name="cyan"><color rgba="0 1.0 1.0 1.0"/></material>
-    <material name="gray"><color rgba="0.5 0.5 0.5 1.0"/></material>
-    <material name="white"><color rgba="1 1 1 1"/></material>
-    <material name="orange"><color rgba="1 0.3 0.1 1"/></material>
-    <material name="blue"><color rgba="0.2 0.2 1 1"/></material>
-    <material name="black"><color rgba="0 0 0 1"/></material>
-    <material name="red"><color rgba="1 0 0 1"/></material>
+    <xacro:property name="caster_wheel_zoff" value="${caster_wheel_radius}"/>
+    <xacro:property name="bumper_thickness" value="0.005"/>
+    <xacro:property name="bumper_length" value="0.05"/>
+    <xacro:property name="bumper_height" value="${chassis_height}"/>
+    <xacro:property name="camera_length" value="0.065"/>
+    <xacro:property name="camera_height" value="0.05"/>
+    <xacro:property name="camera_offset_above_chassis" value="0.025"/>
+    <xacro:property name="camera_overhang" value="0.013"/>
+    <material name="white"><color rgba="1.0 1.0 1.0 1.0"/></material>
+    <material name="adi_blue"><color rgba="0.0 0.32 0.65 1.0"/></material>
+    <material name="gray"><color rgba="0.65 0.65 0.65 1.0"/></material>
+    <material name="black"><color rgba="0.1 0.1 0.1 1.0"/></material>
     <!-- BASE LINK -->
     <link name="${prefix}base_link"></link>
@@ -33,8 +38,8 @@
     </xacro:imu_adis16470>
     <xacro:tof_adtf3175d prefix="${prefix}" parent="${prefix}base_link">
-        <origin xyz="${chassis_length / 2}  0 0.055" rpy="0 0 0" />
+        <origin xyz="${chassis_length/2 + camera_overhang - camera_length/2} 0 ${chassis_clearance_ground + camera_offset_above_chassis + camera_height/2}" rpy="0 0 0" />
     </xacro:tof_adtf3175d>
     <xacro:lidar prefix="${prefix}" parent="${prefix}base_link">
-        <origin xyz="${chassis_length/2} 0 0.055" rpy="0 0 0" />
+        <origin xyz="${chassis_length/2 + camera_overhang - camera_length/2} 0 ${chassis_clearance_ground + camera_offset_above_chassis + camera_height/2}" rpy="0 0 0" />
     </xacro:lidar>
     <!-- BASE_FOOTPRINT LINK -->
@@ -57,5 +62,5 @@
                 <box size="${chassis_length} ${chassis_width} ${chassis_height}"/>
             </geometry>
-            <material name="cyan"/>
+            <material name="white"/>
         </visual>
         <collision>
@@ -70,6 +75,47 @@
     </link>
     <gazebo reference="${prefix}chassis">
-        <material>Gazebo/Gray</material>
+        <material>Gazebo/White</material>
     </gazebo>
+    <!-- CORNER BUMPERS (L-shaped: lateral + front/rear sections) -->
+    <xacro:macro name="corner_bumper" params="name x_reflect y_reflect">
+        <!-- Lateral section (along Y, on the side) -->
+        <joint name="${prefix}${name}_bumper_lat_joint" type="fixed">
+            <parent link="${prefix}chassis"/>
+            <child link="${prefix}${name}_bumper_lat"/>
+            <origin xyz="${x_reflect*(chassis_length/2 - bumper_length/2)} ${y_reflect*(chassis_width/2 + bumper_thickness/2)} ${chassis_zoff}" rpy="0 0 0"/>
+        </joint>
+        <link name="${prefix}${name}_bumper_lat">
+            <visual>
+                <geometry>
+                    <box size="${bumper_length} ${bumper_thickness} ${bumper_height}"/>
+                </geometry>
+                <material name="adi_blue"/>
+            </visual>
+        </link>
+        <gazebo reference="${prefix}${name}_bumper_lat">
+            <material>Gazebo/Blue</material>
+        </gazebo>
+        <!-- Front/rear section (along X, on the front/back) -->
+        <joint name="${prefix}${name}_bumper_front_joint" type="fixed">
+            <parent link="${prefix}chassis"/>
+            <child link="${prefix}${name}_bumper_front"/>
+            <origin xyz="${x_reflect*(chassis_length/2 + bumper_thickness/2)} ${y_reflect*(chassis_width/2 - bumper_length/2 + bumper_thickness/2)} ${chassis_zoff}" rpy="0 0 0"/>
+        </joint>
+        <link name="${prefix}${name}_bumper_front">
+            <visual>
+                <geometry>
+                    <box size="${bumper_thickness} ${bumper_length + bumper_thickness} ${bumper_height}"/>
+                </geometry>
+                <material name="adi_blue"/>
+            </visual>
+        </link>
+        <gazebo reference="${prefix}${name}_bumper_front">
+            <material>Gazebo/Blue</material>
+        </gazebo>
+    </xacro:macro>
+    <xacro:corner_bumper name="front_left" x_reflect="1" y_reflect="1"/>
+    <xacro:corner_bumper name="front_right" x_reflect="1" y_reflect="-1"/>
+    <xacro:corner_bumper name="rear_left" x_reflect="-1" y_reflect="1"/>
+    <xacro:corner_bumper name="rear_right" x_reflect="-1" y_reflect="-1"/>
     <!-- LEFT WHEEL LINK -->
     <joint name="left_wheel_joint" type="continuous">
@@ -84,5 +130,5 @@
                 <cylinder radius="${wheel_radius}" length="${wheel_width}"/>
             </geometry>
-            <material name="blue"/>
+            <material name="gray"/>
         </visual>
         <collision>
@@ -96,5 +142,5 @@
     </link>
     <gazebo reference="${prefix}left_wheel">
-        <material>Gazebo/Black</material>
+        <material>Gazebo/Grey</material>
         <mu1>1.5</mu1> <!-- SLIP_FIX was 2.5 -->
         <mu2>1.5</mu2> <!-- SLIP_FIX was 2.5 -->
@@ -116,5 +162,5 @@
                 <cylinder radius="${wheel_radius}" length="${wheel_width}"/>
             </geometry>
-            <material name="blue"/>
+            <material name="gray"/>
         </visual>
         <collision>
@@ -128,5 +174,5 @@
     </link>
     <gazebo reference="${prefix}right_wheel">
-        <material>Gazebo/Black</material>
+        <material>Gazebo/Grey</material>
         <mu1>1.5</mu1> <!-- SLIP_FIX was 2.5 -->
         <mu2>1.5</mu2> <!-- SLIP_FIX was 2.5 -->
@@ -143,5 +189,5 @@
                     <sphere radius="${caster_wheel_radius}"/>
                 </geometry>
-                <material name="cyan"/>
+                <material name="gray"/>
             </visual>
             <collision>
@@ -161,5 +207,5 @@
         </joint>
         <gazebo reference="${prefix}_link">
-            <material>Gazebo/Blue</material>
+            <material>Gazebo/Grey</material>
             <mu1 value="0.001"/>
             <mu2 value="0.001"/>

Commit message: ad_r1m_gazebo: Migrate simulation from Gazebo Classic 11 to Gazebo Harmonic
Replace all Gazebo Classic dependencies with Gazebo Harmonic (gz-sim 8):
- Sensor xacros: remove libgazebo_ros_* plugins, add <topic> elements
- URDF materials: replace Gazebo/* scripts with RGBA ambient/diffuse/specular
- Friction: wrap shorthand params in proper SDF <surface> blocks
- ros2_control: GazeboSystem -> GazeboSimSystem, plugin -> gz_ros2_control-system
- Worlds: convert empty.world and obstacles.world to SDF 1.9 with gz-sim plugins
- Launch files: gazebo_ros -> ros_gz_sim, add ros_gz_bridge parameter_bridge
- Package deps: gazebo_ros_pkgs -> ros_gz, gazebo_ros2_control -> gz_ros2_control
- Remove Classic-only gazebo_params.yaml

Docker setup added under ad_r1m_examples/imu_hil_demo/ (Dockerfile + entrypoint.sh)
for running the HIL demo with Gazebo Harmonic GUI. gz_ros2_control is built from
source in the container because the apt package links against Fortress (gz-sim6).

Known limitations:
- factory.world and aws_office.world are currently not migrated.
- Downloaded obstacle models (construction_barrel, etc.) may still contain
  Classic material scripts -- geometry works but textures may be missing
- The old .world files are still present and unused

Signed-off-by: Tudor Alinei-Poiana <tudor.alinei-poiana@analog.com>

File: ad_r1m_description/urdf/_imu_adis16470.xacro (robot description, xacro)
@@ -31,14 +31,8 @@
     <gazebo reference="${prefix}imu">
         <sensor name="imu_sensor" type="imu">
-        <plugin filename="libgazebo_ros_imu_sensor.so" name="imu_plugin">
-            <ros>
-            <remapping>~/out:=imu</remapping>
-            </ros>
-            <initial_orientation_as_reference>false</initial_orientation_as_reference>
-            <frame_name>imu</frame_name>
-        </plugin>
         <always_on>true</always_on>
         <update_rate>100</update_rate>
         <visualize>true</visualize>
+        <topic>imu</topic>
         <imu>
             <angular_velocity>

File: ad_r1m_description/urdf/_lidar.xacro (robot description, xacro)
@@ -6,9 +6,10 @@
 <xacro:macro name="lidar" params="prefix parent *origin">
     <gazebo reference="${prefix}cam1_scan">
-        <sensor name="laser" type="ray">
+        <sensor name="laser" type="gpu_lidar">
             <pose>0 0 0 0 0 0</pose>
             <visualize>false</visualize>
             <update_rate>30</update_rate>
-            <ray>
+            <topic>scan</topic>
+            <lidar>
                 <scan>
                     <horizontal>
@@ -22,12 +23,5 @@
                     <max>5.0</max>
                 </range>
-            </ray>
-            <plugin name="laser_controller" filename="libgazebo_ros_ray_sensor.so">
-                <ros>
-                    <remapping>~/out:=scan</remapping>
-                </ros>
-                <output_type>sensor_msgs/LaserScan</output_type>
-                <frame_name>${prefix}cam1_scan</frame_name>
-            </plugin>
+            </lidar>
         </sensor>
     </gazebo>

File: ad_r1m_description/urdf/_tof_adtf3175d.xacro (robot description, xacro)
@@ -49,10 +49,15 @@
     <link name="${prefix}cam1_scan"></link>
     <gazebo reference="${prefix}cam1_adtf31xx">
-        <material>Gazebo/Black</material>
+        <material>
+            <ambient>0.1 0.1 0.1 1</ambient>
+            <diffuse>0.1 0.1 0.1 1</diffuse>
+            <specular>0.1 0.1 0.1 1</specular>
+        </material>
         <!-- 75deg FOV, 512x512, 0.3-5.0m range -->
-        <sensor name="cam1_depth" type="depth">
+        <sensor name="cam1_depth" type="depth_camera">
             <pose>0 0 0 0 0 0</pose>
             <visualize>true</visualize>
             <update_rate>30</update_rate>
+            <topic>cam1</topic>
             <camera>
                 <horizontal_fov>1.309</horizontal_fov>
@@ -72,15 +77,4 @@
                 </noise>
             </camera>
-            <plugin name="depth_camera_controller" filename="libgazebo_ros_camera.so">
-                <camera_name>cam1</camera_name>
-                <frame_name>${prefix}cam1_adtf31xx_optical</frame_name>
-                <min_depth>0.3</min_depth>
-                <max_depth>5.0</max_depth>
-                <ros>
-                    <remapping>cam1/image_raw:=cam1/ab_image</remapping>
-                    <remapping>cam1/depth/image_raw:=cam1/depth_image</remapping>
-                    <remapping>cam1/points:=cam1/point_cloud</remapping>
-                </ros>
-            </plugin>
         </sensor>
     </gazebo>

File: ad_r1m_description/urdf/ad_r1m_base.urdf.xacro (robot description, xacro)
@@ -73,5 +73,9 @@
     </link>
     <gazebo reference="${prefix}chassis">
-        <material>Gazebo/White</material>
+        <material>
+            <ambient>1.0 1.0 1.0 1</ambient>
+            <diffuse>1.0 1.0 1.0 1</diffuse>
+            <specular>1.0 1.0 1.0 1</specular>
+        </material>
     </gazebo>
     <!-- CORNER BUMPERS (L-shaped: lateral + front/rear sections) -->
@@ -92,5 +96,9 @@
         </link>
         <gazebo reference="${prefix}${name}_bumper_lat">
-            <material>Gazebo/Blue</material>
+            <material>
+                <ambient>0.0 0.0 0.8 1</ambient>
+                <diffuse>0.0 0.0 0.8 1</diffuse>
+                <specular>0.0 0.0 0.8 1</specular>
+            </material>
         </gazebo>
         <!-- Front/rear section (along X, on the front/back) -->
@@ -109,5 +117,9 @@
         </link>
         <gazebo reference="${prefix}${name}_bumper_front">
-            <material>Gazebo/Blue</material>
+            <material>
+                <ambient>0.0 0.0 0.8 1</ambient>
+                <diffuse>0.0 0.0 0.8 1</diffuse>
+                <specular>0.0 0.0 0.8 1</specular>
+            </material>
         </gazebo>
     </xacro:macro>
@@ -140,11 +152,15 @@
     </link>
     <gazebo reference="${prefix}left_wheel">
-        <material>Gazebo/Grey</material>
-        <mu1>1.5</mu1> <!-- SLIP_FIX was 2.5 -->
-        <mu2>1.5</mu2> <!-- SLIP_FIX was 2.5 -->
-        <kp>1000000</kp> <!-- SLIP_FIX -->
-        <kd>100</kd> <!-- SLIP_FIX -->
-        <minDepth>0.001</minDepth> <!-- SLIP_FIX -->
-        <maxVel>0.1</maxVel> <!-- SLIP_FIX -->
+        <material>
+            <ambient>0.5 0.5 0.5 1</ambient>
+            <diffuse>0.5 0.5 0.5 1</diffuse>
+            <specular>0.5 0.5 0.5 1</specular>
+        </material>
+        <collision>
+            <surface>
+                <friction><ode><mu>1.5</mu><mu2>1.5</mu2></ode></friction>
+                <contact><ode><kp>1e6</kp><kd>100</kd><min_depth>0.001</min_depth><max_vel>0.1</max_vel></ode></contact>
+            </surface>
+        </collision>
     </gazebo>
     <!-- RIGHT WHEEL LINK -->
@@ -172,11 +188,15 @@
     </link>
     <gazebo reference="${prefix}right_wheel">
-        <material>Gazebo/Grey</material>
-        <mu1>1.5</mu1> <!-- SLIP_FIX was 2.5 -->
-        <mu2>1.5</mu2> <!-- SLIP_FIX was 2.5 -->
-        <kp>1000000</kp> <!-- SLIP_FIX -->
-        <kd>100</kd> <!-- SLIP_FIX -->
-        <minDepth>0.001</minDepth> <!-- SLIP_FIX -->
-        <maxVel>0.1</maxVel> <!-- SLIP_FIX -->
+        <material>
+            <ambient>0.5 0.5 0.5 1</ambient>
+            <diffuse>0.5 0.5 0.5 1</diffuse>
+            <specular>0.5 0.5 0.5 1</specular>
+        </material>
+        <collision>
+            <surface>
+                <friction><ode><mu>1.5</mu><mu2>1.5</mu2></ode></friction>
+                <contact><ode><kp>1e6</kp><kd>100</kd><min_depth>0.001</min_depth><max_vel>0.1</max_vel></ode></contact>
+            </surface>
+        </collision>
     </gazebo>
     <!-- CASTER WHEEL LINKS -->
@@ -205,11 +225,15 @@
         </joint>
         <gazebo reference="${prefix}_link">
-            <material>Gazebo/Grey</material>
-            <mu1 value="0.001"/>
-            <mu2 value="0.001"/>
-            <kp>1000000</kp> <!-- SLIP_FIX -->
-            <kd>100</kd> <!-- SLIP_FIX -->
-            <minDepth>0.001</minDepth> <!-- SLIP_FIX -->
-            <maxVel>0.1</maxVel> <!-- SLIP_FIX -->
+            <material>
+                <ambient>0.5 0.5 0.5 1</ambient>
+                <diffuse>0.5 0.5 0.5 1</diffuse>
+                <specular>0.5 0.5 0.5 1</specular>
+            </material>
+            <collision>
+                <surface>
+                    <friction><ode><mu>0.001</mu><mu2>0.001</mu2></ode></friction>
+                    <contact><ode><kp>1e6</kp><kd>100</kd><min_depth>0.001</min_depth><max_vel>0.1</max_vel></ode></contact>
+                </surface>
+            </collision>
         </gazebo>
     </xacro:macro>

File: ad_r1m_gazebo/urdf/ad_r1m_sim.urdf.xacro (robot description, xacro)
@@ -11,8 +11,7 @@
     <xacro:include filename="$(find ad_r1m_description)/urdf/ad_r1m_base.urdf.xacro" />
     <xacro:ad_r1m_base prefix="${prefix}" use_sim="true" />
-    <!-- Bind gazebo_ros2_control to previously defined joints (e.g. left_wheel_joint) -->
-    <ros2_control name="GazeboSystem" type="system">
+    <ros2_control name="GZSimSystem" type="system">
         <hardware>
-            <plugin>gazebo_ros2_control/GazeboSystem</plugin>
+            <plugin>gz_ros2_control/GazeboSimSystem</plugin>
         </hardware>
         <joint name="left_wheel_joint">
@@ -34,5 +33,5 @@
     </ros2_control>
     <gazebo>
-        <plugin name="gazebo_ros2_control" filename="libgazebo_ros2_control.so">
+        <plugin filename="gz_ros2_control-system" name="gz_ros2_control::GazeboSimROS2ControlPlugin">
             <parameters>$(find ad_r1m_control)/config/controllers.yaml</parameters>
             <parameters>$(find ad_r1m_gazebo)/config/gaz_ros2_ctl_use_sim.yaml</parameters>

File: ad_r1m_perception_cuvslam/urdf/_d435.gazebo.xacro (robot description, xacro)
@@ -86,5 +86,5 @@
           </ros>
           <!-- Tell plugin which TF frame this camera belongs to -->
-          <frame_name>${infrared1_optical_frame}</frame_name>
+          <frame_name>${infrared2_optical_frame}</frame_name>
         </plugin>
       </sensor>
